Commit message: 角度制限を追加

File: erasers_kachaka/erasers_kachaka_manipulation/urdf/manipulation_description.urdf.xacro (robot description, xacro)
@@ -82,9 +82,9 @@
   <xacro:property name="JOINT_VELOCITY_LIMIT" value="4.81710873"/>
   <xacro:property name="JOINT_1_LOWER_LIMIT" value="${radians(-157)}"/>
-  <xacro:property name="JOINT_1_UPPER_LIMIT" value="${radians(157)}"/>
+  <xacro:property name="JOINT_1_UPPER_LIMIT" value="${radians(90)}"/>
   <xacro:property name="JOINT_2_LOWER_LIMIT" value="${radians(-90)}"/>
   <xacro:property name="JOINT_2_UPPER_LIMIT" value="${radians(90)}"/>
-  <xacro:property name="JOINT_3_LOWER_LIMIT" value="${radians(-157)}"/>
-  <xacro:property name="JOINT_3_UPPER_LIMIT" value="${radians(157)}"/>
+  <xacro:property name="JOINT_3_LOWER_LIMIT" value="${radians(-45)}"/>
+  <xacro:property name="JOINT_3_UPPER_LIMIT" value="${radians(45)}"/>
   <!-- JOINT_4はサーボ可動範囲を超えやすいため、LOWER_LIMITをサーボのリミット値より小さくする -->
   <xacro:property name="JOINT_4_LOWER_LIMIT" value="${radians(-159)}"/>
@@ -96,6 +96,6 @@
   <xacro:property name="JOINT_6_LOWER_LIMIT" value="${radians(-90)}"/>
   <xacro:property name="JOINT_6_UPPER_LIMIT" value="${radians(90)}"/>
-  <xacro:property name="JOINT_7_LOWER_LIMIT" value="${radians(-167)}"/>
-  <xacro:property name="JOINT_7_UPPER_LIMIT" value="${radians(167)}"/>
+  <xacro:property name="JOINT_7_LOWER_LIMIT" value="${radians(-90)}"/>
+  <xacro:property name="JOINT_7_UPPER_LIMIT" value="${radians(90)}"/>
   <xacro:property name="JOINT_HAND_LOWER_LIMIT" value="${radians(-5)}"/>
   <xacro:property name="JOINT_HAND_UPPER_LIMIT" value="${radians(90)}"/>
