Commit message: add prefix for container kachaka

File: erasers_kachaka/erasers_kachaka_description/urdf/erasers_kachaka_container_description.urdf.xacro (robot description, xacro)
@@ -2,14 +2,13 @@
 <robot name="erasers_kachaka" xmlns:xacro="http://ros.org/wiki/xacro">
   <xacro:include filename="$(find kachaka_description)/robot/kachaka.urdf.xacro" />
-  <xacro:include filename="$(find kachaka_shelf_description)/urdf/short_shelf_description.urdf.xacro" />
+  <xacro:include filename="$(find kachaka_shelf_description)/urdf/container_description.urdf.xacro" />
   <xacro:include filename="$(find realsense2_description)/urdf/_d435.urdf.xacro" />
   <!-- xacro:include filename="$(find kachaka_shelf_description)/urdf/short_shelf_description.urdf.xacro" /-->
-  <joint name="base_to_shelf" type="fixed">
-    <parent link="base_link" />
-    <child link="shelf_base_link" />
+  <xacro:arg name="robot_name" default="" />
+  <xacro:property name="prefix" value="$(arg robot_name)_" />
+  <joint name="${prefix}base_to_shelf" type="fixed">
+    <parent link="${prefix}base_link" />
+    <child link="${prefix}shelf_base_link" />
     <origin xyz="0 0 0.15" rpy="0 0 0" />
   </joint>
-  <xacro:sensor_d435 parent="shelf_middle_plate_link" name="d435" >
-    <origin xyz="0 0 0.62" rpy="0 0 0"/>
-  </xacro:sensor_d435>
 </robot>

Commit message: problem of container kachaka name space

File: erasers_kachaka/erasers_kachaka_description/urdf/erasers_kachaka_container_description.urdf.xacro (robot description, xacro)
@@ -6,5 +6,5 @@
   <!-- xacro:include filename="$(find kachaka_shelf_description)/urdf/short_shelf_description.urdf.xacro" /-->
   <xacro:arg name="robot_name" default="" />
-  <xacro:property name="prefix" value="$(arg robot_name)_" />
+  <xacro:property name="prefix" value="$(arg robot_name)/" />
   <joint name="${prefix}base_to_shelf" type="fixed">
     <parent link="${prefix}base_link" />
