Commit message: d435 に換装

File: erasers_kachaka/erasers_kachaka_description/urdf/with_piper.urdf.xacro (robot description, xacro)
@@ -3,5 +3,6 @@
   <xacro:include filename="$(find erasers_kachaka_description)/urdf/erasers_kachaka_description.urdf.xacro" />
   <xacro:include filename="$(find erasers_piper_description)/urdf/piper_description.xacro" />
-  <xacro:include filename="$(find depthai_descriptions)/urdf/include/depthai_macro.urdf.xacro" />
+  <!-- xacro:include filename="$(find depthai_descriptions)/urdf/include/depthai_macro.urdf.xacro" /-->
+  <xacro:include filename="$(find realsense2_description)/urdf/_d435.urdf.xacro" />
   <xacro:piper_macro
     use_base="false"
@@ -9,9 +10,12 @@
     x="0.07" y="0" z="0.15"
     roll="0" pitch="0" yaw="0"/>
-  <xacro:depthai_camera camera_name="oak" parent="gripper_base"
+  <!-- xacro:depthai_camera camera_name="oak" parent="gripper_base"
     camera_model="OAK-D-PRO" base_frame="oak-d_frame"
     cam_pos_x="-0.05" cam_pos_y="0.0" cam_pos_z="0.075"
     cam_roll="0.0" cam_pitch="-1.57" cam_yaw="0.0"
     rs_compat="false"
-  />
+  /-->
+  <xacro:sensor_d435 parent="gripper_base" name="arm_camera" >
+     <origin xyz="-0.05 0 0.075" rpy="0 -1.57 0"/>
+  </xacro:sensor_d435>
 </robot>

Commit message: arm camera の位置を微調整

File: erasers_kachaka/erasers_kachaka_description/urdf/with_piper.urdf.xacro (robot description, xacro)
@@ -17,5 +17,5 @@
   /-->
   <xacro:sensor_d435 parent="gripper_base" name="arm_camera" >
-     <origin xyz="-0.05 0 0.075" rpy="0 -1.57 0"/>
+     <origin xyz="-0.03 0 0.06" rpy="0 -1.57 0"/>
   </xacro:sensor_d435>
 </robot>
