Commit message: change shelf distance

File: erasers_kachaka/erasers_kachaka_description/urdf/erasers_kachaka_description.urdf.xacro (robot description, xacro)
@@ -2,9 +2,9 @@
 <robot name="erasers_kachaka" xmlns:xacro="http://ros.org/wiki/xacro">
   <xacro:include filename="$(find kachaka_description)/robot/kachaka.urdf.xacro" />
-  <xacro:include filename="$(find kachaka_shelf_description)/urdf/shelf_description.urdf.xacro" />
+  <xacro:include filename="$(find kachaka_shelf_description)/urdf/short_shelf_description.urdf.xacro" />
   <joint name="docking_to_shelf" type="fixed">
     <parent link="docking_link" />
     <child link="shelf_base_link" />
-    <origin xyz="0 0 0.1" rpy="0 0 0" />
+    <origin xyz="0 0 0.15" rpy="0 0 0" />
   </joint>
 </robot>

Commit message: change link docking to base_link

File: erasers_kachaka/erasers_kachaka_description/urdf/erasers_kachaka_description.urdf.xacro (robot description, xacro)
@@ -4,6 +4,6 @@
   <xacro:include filename="$(find kachaka_shelf_description)/urdf/shelf_description.urdf.xacro" />
   <!-- xacro:include filename="$(find kachaka_shelf_description)/urdf/short_shelf_description.urdf.xacro" /-->
-  <joint name="docking_to_shelf" type="fixed">
-    <parent link="docking_link" />
+  <joint name="base_to_shelf" type="fixed">
+    <parent link="base_link" />
     <child link="shelf_base_link" />
     <origin xyz="0 0 0.15" rpy="0 0 0" />

Commit message: edit  urdf

File: erasers_kachaka/erasers_kachaka_description/urdf/erasers_kachaka_description.urdf.xacro (robot description, xacro)
@@ -9,3 +9,8 @@
     <origin xyz="0 0 0.15" rpy="0 0 0" />
   </joint>
+  <joint name="camera_joint" type="fixed">
+      <origin xyz="0.0 0.00 0.49" rpy="0 0 0" />
+      <parent link="base_link"/>
+      <child link="camera_link" />
+  </joint>
 </robot>

File: erasers_kachaka/erasers_kachaka_description/urdf/with_piper.urdf.xacro (robot description, xacro)
@@ -15,5 +15,5 @@
     cam_roll="0.0" cam_pitch="-1.57" cam_yaw="0.0"
     rs_compat="false"
-  /-->
+  / -->
   <xacro:sensor_d435 parent="gripper_base" name="arm_camera" >
      <origin xyz="-0.05 0 0.075" rpy="0 -1.57 0"/>

Commit message: Fix camera TF name

File: erasers_kachaka/erasers_kachaka_description/urdf/erasers_kachaka_description.urdf.xacro (robot description, xacro)
@@ -1,7 +1,13 @@
 <?xml version="1.0" ?>
 <robot name="erasers_kachaka" xmlns:xacro="http://ros.org/wiki/xacro">
-  <xacro:include filename="$(find kachaka_description)/robot/kachaka.urdf.xacro" />
+  <xacro:include filename="$(find erasers_kachaka_description)/urdf/_kachaka.urdf.xacro" />
+  <xacro:include filename="$(find kachaka_description)/urdf/_materials.urdf.xacro" />
+  <xacro:include filename="$(find kachaka_description)/urdf/_values.urdf.xacro" />
   <xacro:include filename="$(find kachaka_shelf_description)/urdf/shelf_description.urdf.xacro" />
   <!-- xacro:include filename="$(find kachaka_shelf_description)/urdf/short_shelf_description.urdf.xacro" /-->
+  <link name="base_footprint" />
+  <xacro:kachaka_robot parent="base_footprint">
+    <origin xyz="0 0 0" rpy="0 0 0"/>
+  </xacro:kachaka_robot>
   <joint name="base_to_shelf" type="fixed">
     <parent link="base_link" />
