Commit message: Support ToF camera

File: erasers_kachaka/erasers_kachaka_description/urdf/_kachaka.urdf.xacro (robot description, xacro)
@@ -144,9 +144,9 @@
           type="fixed">
       <parent link="base_link" />
-      <child link="tof_link" />
+      <child link="tof_camera" />
       <origin rpy="-${PI / 4.0} 0 -${PI / 2.0}"
               xyz="0.221 0.0 0.0418" />
     </joint>
-    <link name="tof_link" />
+    <link name="tof_camera" />
     <!-- Docking -->
     <joint name="docking_joint"
