Commit message: adjuest robot description

File: erasers_kachaka/erasers_kachaka_description/urdf/opl_shelf.urdf.xacro (robot description, xacro)
@@ -47,5 +47,5 @@
     <parent link="shelf_base_link"/>
     <child link="shelf_middle_plate_link"/>
-    <origin xyz="0 0 ${shelf_distance_short}"/> <!-- Z軸方向に0.15m上 -->
+    <origin xyz="0 0 ${shelf_distance_long}"/> <!-- Z軸方向に0.15m上 -->
   </joint>
 </robot>
